File: Nes Sound Expansion OPNA 4016/Nes Sound Expansion.sch (KiCad schematic (older format))
At the start: 41 parts, among them J1 NES-SNES Port1, J2 NES-SNES Port2, J3 EXP 1-24, J4 EXP 25-48, J5 EN Switch, J6 AudioJack2_Ground_Switch, J7 EN LED, U1 74LS139, U10 74LS257, U2 74LS132, U6 74LS174, U7 74LS174, U8 74LS257, U9 74LS257, X1 CXO_DIP8

Commit message: Fixed floating signals and famicom exp audio
Addressing issues caused by floating signals when a cart without hardware addressing is used
Added famicom expansion resistors to all 3 popular EXP pins.
Parts:
- added R16, R17: 1k, Resistor_SMD:R_0805_2012Metric_Pad1.20x1.40mm_HandSolder, symbol Device:R
- added R? (x2): 47k, Resistor_SMD:R_0805_2012Metric_Pad1.20x1.40mm_HandSolder, symbol Device:R
- R5, R8: value 1k -> 600Ω
- R6, R7: value 1k -> 3k
Connections:
- wire segments 107 -> 118
Changed lines of the file:
@@
 P 8750 2500
 F 0 "R5" V 8543 2500 50  0000 C CNN
-F 1 "1k" V 8634 2500 50  0000 C CNN
+F 1 "600Ω" V 8634 2500 50  0000 C CNN
 F 2 "Resistor_SMD:R_0805_2012Metric_Pad1.20x1.40mm_HandSolder" V 8680 2500 50  0001 C CNN
 F 3 "~" H 8750 2500 50  0001 C CNN
@@
 P 8750 2900
 F 0 "R6" V 8543 2900 50  0000 C CNN
-F 1 "1k" V 8634 2900 50  0000 C CNN
+F 1 "3k" V 8634 2900 50  0000 C CNN
 F 2 "Resistor_SMD:R_0805_2012Metric_Pad1.20x1.40mm_HandSolder" V 8680 2900 50  0001 C CNN
 F 3 "~" H 8750 2900 50  0001 C CNN
@@
 P 8750 3350
 F 0 "R7" V 8543 3350 50  0000 C CNN
-F 1 "1k" V 8634 3350 50  0000 C CNN
+F 1 "3k" V 8634 3350 50  0000 C CNN
 F 2 "Resistor_SMD:R_0805_2012Metric_Pad1.20x1.40mm_HandSolder" V 8680 3350 50  0001 C CNN
 F 3 "~" H 8750 3350 50  0001 C CNN
@@
 P 8750 3850
 F 0 "R8" V 8543 3850 50  0000 C CNN
-F 1 "1k" V 8634 3850 50  0000 C CNN
+F 1 "600Ω" V 8634 3850 50  0000 C CNN
 F 2 "Resistor_SMD:R_0805_2012Metric_Pad1.20x1.40mm_HandSolder" V 8680 3850 50  0001 C CNN
 F 3 "~" H 8750 3850 50  0001 C CNN
@@
 	0    1    1    0
 $EndComp
+$Comp
+L Device:R R16
+U 1 1 60948AFF
+P 900 3250
+F 0 "R16" V 693 3250 50  0000 C CNN
+F 1 "1k" V 784 3250 50  0000 C CNN
+F 2 "Resistor_SMD:R_0805_2012Metric_Pad1.20x1.40mm_HandSolder" V 830 3250 50  0001 C CNN
+F 3 "~" H 900 3250 50  0001 C CNN
+	1    900  3250
+	0    1    1    0
+$EndComp
+$Comp
+L Device:R R17
+U 1 1 60949AED
+P 900 3400
+F 0 "R17" V 693 3400 50  0000 C CNN
+F 1 "1k" V 784 3400 50  0000 C CNN
+F 2 "Resistor_SMD:R_0805_2012Metric_Pad1.20x1.40mm_HandSolder" V 830 3400 50  0001 C CNN
+F 3 "~" H 900 3400 50  0001 C CNN
+	1    900  3400
+	0    1    1    0
+$EndComp
+$Comp
+L power:GND #PWR0132
+U 1 1 6094A089
+P 1050 3250
+F 0 "#PWR0132" H 1050 3000 50  0001 C CNN
+F 1 "GND" H 1055 3077 50  0000 C CNN
+F 2 "" H 1050 3250 50  0001 C CNN
+F 3 "" H 1050 3250 50  0001 C CNN
+	1    1050 3250
+	0    -1   -1   0
+$EndComp
+$Comp
+L power:GND #PWR0133
+U 1 1 6094AAFB
+P 1050 3400
+F 0 "#PWR0133" H 1050 3150 50  0001 C CNN
+F 1 "GND" H 1055 3227 50  0000 C CNN
+F 2 "" H 1050 3400 50  0001 C CNN
+F 3 "" H 1050 3400 50  0001 C CNN
+	1    1050 3400
+	0    -1   -1   0
+$EndComp
+Text GLabel 750  3250 0    50   Input ~ 0
+A14
+Text GLabel 750  3400 0    50   Input ~ 0
+A13
+$Comp
+L Device:R R?
+U 1 1 6097469C
+P 1500 1300
+F 0 "R?" V 1293 1300 50  0000 C CNN
+F 1 "47k" V 1384 1300 50  0000 C CNN
+F 2 "Resistor_SMD:R_0805_2012Metric_Pad1.20x1.40mm_HandSolder" V 1430 1300 50  0001 C CNN
+F 3 "~" H 1500 1300 50  0001 C CNN
+	1    1500 1300
+	-1   0    0    1
+$EndComp
+$Comp
+L Device:R R?
+U 1 1 6097489A
+P 1400 1300
+F 0 "R?" V 1193 1300 50  0000 C CNN
+F 1 "47k" V 1284 1300 50  0000 C CNN
+F 2 "Resistor_SMD:R_0805_2012Metric_Pad1.20x1.40mm_HandSolder" V 1330 1300 50  0001 C CNN
+F 3 "~" H 1400 1300 50  0001 C CNN
+	1    1400 1300
+	-1   0    0    1
+$EndComp
+Wire Wire Line
+	1600 1100 1500 1100
+Wire Wire Line
+	1500 1100 1500 1150
+Connection ~ 1600 1100
+Wire Wire Line
+	1500 1100 1400 1100
+Wire Wire Line
+	1400 1100 1400 1150
+Connection ~ 1500 1100
+Wire Wire Line
+	1500 1450 1500 1750
+Wire Wire Line
+	1500 1750 2400 1750
+Wire Wire Line
+	2400 1750 2400 1700
+Wire Wire Line
+	1400 1450 1400 1550
+Wire Wire Line
+	1400 1550 1750 1550
+Wire Wire Line
+	1750 1550 1750 1400
+Wire Wire Line
+	1750 1400 2000 1400
 $EndSCHEMATC

Commit message: minor update
Parts:
- gave numbers to parts that had none: 2
Changed lines of the file:
@@
 A13
 $Comp
-L Device:R R?
+L Device:R R19
 U 1 1 6097469C
 P 1500 1300
-F 0 "R?" V 1293 1300 50  0000 C CNN
+F 0 "R19" V 1293 1300 50  0000 C CNN
 F 1 "47k" V 1384 1300 50  0000 C CNN
 F 2 "Resistor_SMD:R_0805_2012Metric_Pad1.20x1.40mm_HandSolder" V 1430 1300 50  0001 C CNN
@@
 $EndComp
 $Comp
-L Device:R R?
+L Device:R R18
 U 1 1 6097489A
 P 1400 1300
-F 0 "R?" V 1193 1300 50  0000 C CNN
+F 0 "R18" V 1193 1300 50  0000 C CNN
 F 1 "47k" V 1284 1300 50  0000 C CNN
 F 2 "Resistor_SMD:R_0805_2012Metric_Pad1.20x1.40mm_HandSolder" V 1330 1300 50  0001 C CNN

Commit message: Added IRQ from the YMF288
Connections:
- net labels added: IRQ, NMI
Changed lines of the file:
@@
 Wire Wire Line
 	1750 1400 2000 1400
+Text GLabel 2000 1200 0    50   Input ~ 0
+NMI
+Text GLabel 2000 2200 0    50   Input ~ 0
+IRQ
+Text GLabel 4500 3500 2    50   Input ~ 0
+IRQ
 $EndSCHEMATC

Commit message: Added logo, 3.5mm 3d module, removed unused stuff
Parts:
- removed R11: 1k, Resistor_SMD:R_0805_2012Metric_Pad1.20x1.40mm_HandSolder, symbol Device:R
- BU9480F1: footprint Package_SO:SOIC-8_5.275x5.275mm_P1.27mm -> Package_SO:SOIC-8_3.9x4.9mm_P1.27mm
- C1, C3, C4, C5: footprint Capacitor_SMD:C_0504_1310Metric_Pad0.83x1.28mm_HandSolder -> Capacitor_SMD:C_0805_2012Metric
- C10, C11, C12, C13: value 4.7u -> 10uF
- C2: value 10u -> 10uF
- J5: footprint Connector_PinHeader_2.54mm:PinHeader_1x02_P2.54mm_Vertical -> Button_Switch_SMD:SW_DIP_SPSTx01_Slide_6.7x4.1mm_W6.73mm_P2.54mm_LowProfile_JPin; symbol Connector:Conn_01x02_Male -> Switch:SW_SPST
- J7: footprint Connector_PinHeader_2.54mm:PinHeader_1x02_P2.54mm_Vertical -> LED_SMD:LED_0805_2012Metric; symbol Connector:Conn_01x02_Male -> Device:LED
- R1, R10, R12, R13, R14, R16, R17, R18, R19, R2, R3, R4, R6, R7, R9: footprint Resistor_SMD:R_0805_2012Metric_Pad1.20x1.40mm_HandSolder -> Resistor_SMD:R_0805_2012Metric
- R5, R8: value 600Ω -> 560; footprint Resistor_SMD:R_0805_2012Metric_Pad1.20x1.40mm_HandSolder -> Resistor_SMD:R_0805_2012Metric
- U1: value 74LS139 -> 74HC139D
- U10, U8, U9: value 74LS257 -> 74HC257D
- U2: value 74LS132 -> 74HC132D
- U6, U7: value 74LS174 -> 74HC174D
- X1: footprint Oscillator:Oscillator_SMD_SeikoEpson_SG8002CA-4Pin_7.0x5.0mm_HandSoldering -> Oscillator:Oscillator_SMD_SeikoEpson_SG8002CE-4Pin_3.2x2.5mm
